Commit message: launch configuration

File: description/ros2_control/diffbot.ros2_control.xacro (robot description, xacro)
@@ -2,5 +2,33 @@
 <robot xmlns:xacro="http://www.ros.org/wiki/xacro">
   <xacro:macro name="diffbot_ros2_control" params="name prefix">
-    <ros2_control name="${name}" type="system">
+     <ros2_control name="GazeboSystem" type="system">
+            <hardware>
+                <plugin>gazebo_ros2_control/GazeboSystem</plugin>
+            </hardware>
+            <joint name="left_wheel_joint">
+                <command_interface name="velocity">
+                    <param name="min">-10</param>
+                    <param name="max">10</param>
+                </command_interface>
+                <state_interface name="velocity"/>
+                <state_interface name="position"/>
+            </joint>
+            <joint name="right_wheel_joint">
+                <command_interface name="velocity">
+                    <param name="min">-10</param>
+                    <param name="max">10</param>
+                </command_interface>
+                <state_interface name="velocity"/>
+                <state_interface name="position"/>
+            </joint>
+        </ros2_control>
+    </xacro:if>
+    <gazebo>
+        <plugin name="gazebo_ros2_control" filename="libgazebo_ros2_control.so">
+            <parameters>$(find gazebo_control)/config/my_controllers.yaml</parameters>
+            <parameters>$(find gazebo_control)/config/gaz_ros2_ctl_use_sim.yaml</parameters>
+        </plugin>
+    </gazebo>
+    <!-- <ros2_control name="${name}" type="system">
       <hardware>
         <plugin>gazebo_control/DiffDriveArduinoHardware</plugin>
@@ -27,5 +55,5 @@
         <state_interface name="velocity"/>
       </joint>
-    </ros2_control>
+    </ros2_control> -->
   </xacro:macro>
 </robot>

File: description/urdf/diffbot.urdf.xacro (robot description, xacro)
@@ -4,4 +4,5 @@
   <xacro:arg name="prefix" default="" />
   <xacro:include filename="$(find gazebo_control)/urdf/diffbot_description.urdf.xacro" />
+  <xacro:include filename="$(find gazebo_control)/urdf/gazebo_control.xacro" />
   <!-- Import Rviz colors -->
   <xacro:include filename="$(find gazebo_control)/urdf/diffbot.materials.xacro" />

File: description/urdf/diffbot_description.urdf.xacro (robot description, xacro)
@@ -2,41 +2,42 @@
 <robot xmlns:xacro="http://www.ros.org/wiki/xacro">
   <xacro:macro name="diffbot" params="prefix">
-  <xacro:include filename="inertial_macros.xacro"/>
-  <!-- Constants for robot dimensions -->
-  <xacro:property name="PI" value="3.1415926535897931"/>
-  <xacro:property name="base_mass" value="0.3" /> <!-- arbitrary value for base mass -->
-  <xacro:property name="base_width" value="0.5" />
-  <xacro:property name="base_length" value="0.4" />
-  <xacro:property name="base_height" value="0.26" />
-  <xacro:property name="wheel_mass" value="0.3" /> <!-- arbitrary value for wheel mass -->
-  <xacro:property name="wheel_len" value="0.03" />
-  <xacro:property name="wheel_radius" value="0.1" />
-  <xacro:property name="caster_wheel_mass" value="0.1" /> <!-- arbitrary value for caster wheel mass -->
-  <xacro:property name="caster_wheel_radius" value="0.04" />
-  <xacro:property name="z_offset" value="-${base_height/2}" /> <!-- Space btw top of beam and the each joint -->
-  <!-- Base Link -->
-  <link name="${prefix}base_link">
-    <collision>
-      <origin xyz="0 0 0.17" rpy="0 0 1.57"/>
-      <geometry>
-        <box size="${base_width} ${base_length} ${base_height}"/>
-      </geometry>
-    </collision>
-    <visual>
-      <origin xyz="0 0 0.18" rpy="0 0 0"/>
-      <geometry>
-        <box size="${base_width} ${base_length} ${base_height}"/>
-      </geometry>
-      <material name="orange"/>
-    </visual>
-    <inertial>
-      <origin xyz="0 0 0" rpy="0 0 0"/>
-      <mass value="${base_mass}"/>
-      <inertia
-        ixx="${base_mass / 12.0 * (base_length*base_length + base_height*base_height)}" ixy="0.0" ixz="0.0"
-        iyy="${base_mass / 12.0 * (base_height*base_height + base_width*base_width)}" iyz="0.0"
-        izz="${base_mass / 12.0 * (base_width*base_width + base_length*base_length)}"/>
-      </inertial>
-    </link>
+    <xacro:include filename="inertial_macros.xacro"/>
+    <!-- Constants for robot dimensions -->
+    <xacro:property name="PI" value="3.1415926535897931"/>
+    <xacro:property name="base_mass" value="0.3"/>
+    <xacro:property name="base_width" value="0.5"/>
+    <xacro:property name="base_length" value="0.4"/>
+    <xacro:property name="base_height" value="0.26"/>
+    <xacro:property name="wheel_mass" value="0.3"/>
+    <xacro:property name="wheel_len" value="0.03"/>
+    <xacro:property name="wheel_radius" value="0.1"/>
+    <xacro:property name="caster_wheel_mass" value="0.1"/>
+    <xacro:property name="caster_wheel_radius" value="0.04"/>
+    <xacro:property name="z_offset" value="-${base_height/2}"/>
+    <!-- Base Link -->
+    <link name="${prefix}base_link">
+      <collision>
+        <origin xyz="0 0 0.17" rpy="0 0 1.57"/>
+        <geometry>
+          <box size="${base_width} ${base_length} ${base_height}"/>
+        </geometry>
+      </collision>
+      <visual>
+        <origin xyz="0 0 0.18" rpy="0 0 0"/>
+        <geometry>
+          <box size="${base_width} ${base_length} ${base_height}"/>
+        </geometry>
+        <material name="orange"/>
+      </visual>
+      <inertial>
+        <origin xyz="0 0 0" rpy="0 0 0"/>
+        <mass value="${base_mass}"/>
+        <inertia
+          ixx="${base_mass / 12.0 * (base_length*base_length + base_height*base_height)}" ixy="0.0" ixz="0.0"
+          iyy="${base_mass / 12.0 * (base_height*base_height + base_width*base_width)}" iyz="0.0"
+          izz="${base_mass / 12.0 * (base_width*base_width + base_length*base_length)}"/>
+      </inertial>
+    </link>
+    <!-- Left Wheel Joint and Link -->
     <joint name="${prefix}left_wheel_joint" type="continuous">
       <parent link="${prefix}base_link"/>
@@ -46,5 +47,4 @@
       <dynamics damping="0.2"/>
     </joint>
-    <!-- left wheel Link -->
     <link name="${prefix}left_wheel">
       <collision>
@@ -68,6 +68,10 @@
           iyy="${wheel_mass / 12.0 * wheel_radius*wheel_radius}" iyz="0.0"
           izz="${wheel_mass / 12.0 * wheel_radius*wheel_radius}"/>
-        </inertial>
-      </link>
+      </inertial>
+    </link>
+    <gazebo reference="left_wheel">
+      <material>Gazebo/Blue</material>
+    </gazebo>
+    <!-- Right Wheel Joint and Link -->
     <joint name="${prefix}right_wheel_joint" type="continuous">
       <parent link="${prefix}base_link"/>
@@ -77,5 +81,4 @@
       <dynamics damping="0.2"/>
     </joint>
-    <!-- right wheel Link -->
     <link name="${prefix}right_wheel">
       <collision>
@@ -99,6 +102,10 @@
           iyy="${wheel_mass / 12.0 * wheel_radius*wheel_radius}" iyz="0.0"
           izz="${wheel_mass / 12.0 * wheel_radius*wheel_radius}"/>
-        </inertial>
-      </link>
+      </inertial>
+    </link>
+    <gazebo reference="right_wheel">
+      <material>Gazebo/Blue</material>
+    </gazebo>
+    <!-- Caster Wheels -->
     <joint name="${prefix}caster_frontal_wheel_joint" type="fixed">
       <parent link="${prefix}base_link"/>
@@ -106,5 +113,4 @@
       <origin xyz="${base_width/2 - caster_wheel_radius} 0 0.04" rpy="0 0 0"/>
     </joint>
-    <!-- caster frontal wheel Link -->
     <link name="${prefix}caster_frontal_wheel">
       <collision>
@@ -128,6 +134,6 @@
           iyy="${caster_wheel_mass * 0.4 * (caster_wheel_radius * caster_wheel_radius)}" iyz="0.0"
           izz="${caster_wheel_mass * 0.4 * (caster_wheel_radius * caster_wheel_radius)}"/>
-        </inertial>
-      </link>
+      </inertial>
+    </link>
     <joint name="${prefix}caster_rear_wheel_joint" type="fixed">
       <parent link="${prefix}base_link"/>
@@ -135,5 +141,4 @@
       <origin xyz="${-base_width/2 + caster_wheel_radius} 0 0.04" rpy="0 0 0"/>
     </joint>
-    <!-- caster rear wheel Link -->
     <link name="${prefix}caster_rear_wheel">
       <collision>
@@ -157,66 +162,76 @@
           iyy="${caster_wheel_mass * 0.4 * (caster_wheel_radius * caster_wheel_radius)}" iyz="0.0"
           izz="${caster_wheel_mass * 0.4 * (caster_wheel_radius * caster_wheel_radius)}"/>
-        </inertial>
-      </link>
-      <!-- Face Link -->
-      <joint name="face_joint" type="fixed">
-        <parent link="${prefix}base_link"/>
-        <child link="face_link"/>
-        <origin xyz="${base_width/2} 0 ${base_width/2.5}" rpy="0 0 0"/>
+      </inertial>
+    </link>
+    <gazebo reference="caster_frontal_wheel">
+      <material>Gazebo/White</material>
+      <mu1 value="0.001"/>
+      <mu2 value="0.001"/>
+    </gazebo>
+    <gazebo reference="caster_rear_wheel">
+      <material>Gazebo/White</material>
+      <mu1 value="0.001"/>
+      <mu2 value="0.001"/>
+    </gazebo>
+    <!-- Face Link -->
+    <joint name="face_joint" type="fixed">
+      <parent link="${prefix}base_link"/>
+      <child link="face_link"/>
+      <origin xyz="${base_width/2} 0 ${base_width/2.5}" rpy="0 0 0"/>
     </joint>
     <link name="face_link">
-        <visual>
-            <origin xyz="0 0.05 0.01" rpy="0 ${pi/2} 0"/>
-            <geometry>
-                <cylinder radius="0.01" length="0.002"/>
-            </geometry>
-            <material name="black"/>
-        </visual>
-        <visual>
-            <origin xyz="0 -0.05 0.01" rpy="0 ${pi/2} 0"/>
-            <geometry>
-                <cylinder radius="0.01" length="0.002"/>
-            </geometry>
-            <material name="black"/>
-        </visual>
-        <visual>
-            <origin xyz="-0.011 0 -0.00" rpy="0 ${1.5} 0"/>
-            <geometry>
-                <cylinder radius="0.05" length="0.02"/>
-            </geometry>
-            <material name="red"/>
-        </visual>
+      <visual>
+        <origin xyz="0 0.05 0.01" rpy="0 ${pi/2} 0"/>
+        <geometry>
+          <cylinder radius="0.01" length="0.002"/>
+        </geometry>
+        <material name="black"/>
+      </visual>
+      <visual>
+        <origin xyz="0 -0.05 0.01" rpy="0 ${pi/2} 0"/>
+        <geometry>
+          <cylinder radius="0.01" length="0.002"/>
+        </geometry>
+        <material name="black"/>
+      </visual>
+      <visual>
+        <origin xyz="-0.011 0 -0.00" rpy="0 ${1.5} 0"/>
+        <geometry>
+          <cylinder radius="0.05" length="0.02"/>
+        </geometry>
+        <material name="red"/>
+      </visual>
     </link>
     <gazebo reference="face_link">
-        <material>Gazebo/Black</material>
+      <material>Gazebo/Black</material>
     </gazebo>
     <!-- Laser Link -->
     <joint name="laser_joint" type="fixed">
-        <parent link="${prefix}base_link"/>
-        <child link="laser_frame"/>
-        <origin xyz="0.15 0 0.336" rpy="0 0 0"/>
+      <parent link="${prefix}base_link"/>
+      <child link="laser_frame"/>
+      <origin xyz="0.15 0 0.336" rpy="0 0 0"/>
     </joint>
     <link name="laser_frame">
-        <visual>
-            <geometry>
-                <cylinder radius="0.05" length="0.04"/>
-            </geometry>
-            <material name="black"/>
-        </visual>
-        <visual>
-            <origin xyz="0 0 -0.05"/>
-            <geometry>
-                <cylinder radius="0.01" length="0.1"/>
-            </geometry>
-            <material name="black"/>
-        </visual>
-        <collision>
-            <geometry>
-                <cylinder radius="0.05" length="0.04"/>
-            </geometry>
-        </collision>
-        <xacro:inertial_cylinder mass="0.1" length="0.04" radius="0.05">
-            <origin xyz="0 0 0" rpy="0 0 0"/>
-        </xacro:inertial_cylinder>
+      <visual>
+        <geometry>
+          <cylinder radius="0.05" length="0.04"/>
+        </geometry>
+        <material name="black"/>
+      </visual>
+      <visual>
+        <origin xyz="0 0 -0.05"/>
+        <geometry>
+          <cylinder radius="0.01" length="0.1"/>
+        </geometry>
+        <material name="black"/>
+      </visual>
+      <collision>
+        <geometry>
+          <cylinder radius="0.05" length="0.04"/>
+        </geometry>
+      </collision>
+      <xacro:inertial_cylinder mass="0.1" length="0.04" radius="0.05">
+        <origin xyz="0 0 0" rpy="0 0 0"/>
+      </xacro:inertial_cylinder>
     </link>
   </xacro:macro>
